File: Final Report/PCB/pcbcomplete/flyback.kicad_pcb (KiCad board)
At the start: 2 copper layers, 121.9 x 81.3 mm, 31 parts, among them J1 Conn_01x02, J2 Conn_01x02, M1 MNMOS, T1 Transformer_1P_2S, U1 SFH617A-1, U2 UCC28740, U3 TL431LP

Commit message: final additions
pcb design revisited, gerber files, 3D views generated, images are added, final additions to the report
Routing:
- net Net-(D3-Pad2): track 73.7 -> 69.1 mm
