File: Final Report/PCB/pcbcomplete/flyback.sch (KiCad schematic (older format))
At the start: 31 parts, among them J1 Conn_01x02, J2 Conn_01x02, M1 MNMOS, T1 Transformer_1P_2S, U1 SFH617A-1, U2 UCC28740, U3 TL431LP

Commit message: final additions
pcb design revisited, gerber files, 3D views generated, images are added, final additions to the report
Other:
- moved on the sheet: Ccs1, HS1, J1, J2, U2
Changed lines of the file:
@@
 L power:+48V #PWR0101
 U 1 1 5ED3996D
-P 850 2150
-F 0 "#PWR0101" H 850 2000 50  0001 C CNN
-F 1 "+48V" H 865 2323 50  0000 C CNN
-F 2 "" H 850 2150 50  0001 C CNN
-F 3 "" H 850 2150 50  0001 C CNN
-	1    850  2150
+P 2550 3400
+F 0 "#PWR0101" H 2550 3250 50  0001 C CNN
+F 1 "+48V" H 2565 3573 50  0000 C CNN
+F 2 "" H 2550 3400 50  0001 C CNN
+F 3 "" H 2550 3400 50  0001 C CNN
+	1    2550 3400
 	1    0    0    -1
 $EndComp
@@
 L power:GND #PWR0102
 U 1 1 5ED399AD
-P 850 2250
-F 0 "#PWR0102" H 850 2000 50  0001 C CNN
-F 1 "GND" H 855 2077 50  0000 C CNN
-F 2 "" H 850 2250 50  0001 C CNN
-F 3 "" H 850 2250 50  0001 C CNN
-	1    850  2250
-	1    0    0    -1
-$EndComp
-Wire Wire Line
-	850  2150 950  2150
-Wire Wire Line
-	850  2250 950  2250
-Text Label 850  2150 2    50   ~ 0
+P 2550 3500
+F 0 "#PWR0102" H 2550 3250 50  0001 C CNN
+F 1 "GND" H 2555 3327 50  0000 C CNN
+F 2 "" H 2550 3500 50  0001 C CNN
+F 3 "" H 2550 3500 50  0001 C CNN
+	1    2550 3500
+	1    0    0    -1
+$EndComp
+Wire Wire Line
+	2550 3400 2650 3400
+Wire Wire Line
+	2550 3500 2650 3500
+Text Label 2550 3400 2    50   ~ 0
 Vin
-Text Label 850  2250 2    50   ~ 0
+Text Label 2550 3500 2    50   ~ 0
 GND
-Text Label 950  1500 2    50   ~ 0
+Text Label 2650 2750 2    50   ~ 0
 Vout+
-Text Label 950  1600 2    50   ~ 0
+Text Label 2650 2850 2    50   ~ 0
 Vout-
 $Comp
@@
 Wire Wire Line
 	2100 5250 2100 5350
-Text Label 2100 5350 2    50   ~ 0
-GND
-Text Label 3150 5850 3    50   ~ 0
-GND
 Wire Wire Line
 	3150 4850 3150 5100
@@
 Text Label 3700 2850 2    50   ~ 0
 Vin
-Text Label 4700 5900 3    50   ~ 0
+Text Label 4700 5250 3    50   ~ 0
 GND
 Wire Wire Line
@@
 L uccalike:NCP1207B U2
 U 1 1 5EFC2470
-P 4350 5350
-F 0 "U2" H 4350 5817 50  0000 C CNN
-F 1 "UCC28740" H 4350 5726 50  0000 C CNN
-F 2 "Package_SO:SOIC-8-N7_3.9x4.9mm_P1.27mm" H 4350 6000 50  0001 C CIN
-F 3 "http://www.onsemi.com/pub/Collateral/NCP1207B.PDF" H 4350 5350 50  0001 C CNN
-	1    4350 5350
-	1    0    0    -1
-$EndComp
-Wire Wire Line
-	4050 5450 4000 5450
-Wire Wire Line
-	4000 5450 4000 5550
-$Comp
-L power:GND #PWR0113
-U 1 1 5EFC6B08
-P 4050 5600
-F 0 "#PWR0113" H 4050 5350 50  0001 C CNN
-F 1 "GND" H 4055 5427 50  0000 C CNN
-F 2 "" H 4050 5600 50  0001 C CNN
-F 3 "" H 4050 5600 50  0001 C CNN
-	1    4050 5600
-	1    0    0    -1
-$EndComp
-Wire Wire Line
-	4650 5600 4700 5600
-Wire Wire Line
-	4700 4750 4700 5600
-Wire Wire Line
-	4650 3350 4300 3350
-Connection ~ 4300 3350
-Wire Wire Line
-	4300 3350 4300 2900
-Wire Wire Line
-	4050 5150 3800 5150
-Wire Wire Line
-	3800 5150 3800 4300
+P 4350 4600
+F 0 "U2" H 4350 5067 50  0000 C CNN
+F 1 "UCC28740" H 4350 4976 50  0000 C CNN
+F 2 "Package_SO:SOIC-8-N7_3.9x4.9mm_P1.27mm" H 4350 5250 50  0001 C CIN
+F 3 "http://www.onsemi.com/pub/Collateral/NCP1207B.PDF" H 4350 4600 50  0001 C CNN
+	1    4350 4600
+	1    0    0    -1
+$EndComp
+Wire Wire Line
+	4700 4750 4700 4850
 Connection ~ 3800 4300
 Wire Wire Line
 	3800 4300 3150 4300
 Wire Wire Line
-	4100 5300 4050 5300
-Wire Wire Line
-	4050 5300 3850 5300
-Wire Wire Line
-	3850 5300 3850 4950
-Connection ~ 4050 5300
-Wire Wire Line
 	4300 4050 4650 4050
 Wire Wire Line
-	4300 4050 4300 3350
-Wire Wire Line
-	4650 5450 4800 5450
-Wire Wire Line
-	4800 5450 4800 4400
-Wire Wire Line
-	4650 4050 4650 5150
+	4650 4050 4650 4400
 $Comp
 L Device:C Ccs1
 U 1 1 5ED746E5
-P 4700 5750
-F 0 "Ccs1" H 4815 5796 50  0000 L CNN
-F 1 "C" H 4815 5705 50  0000 L CNN
-F 2 "Capacitor_SMD:C_0402_1005Metric" H 4738 5600 50  0001 C CNN
-F 3 "~" H 4700 5750 50  0001 C CNN
-	1    4700 5750
+P 4700 5100
+F 0 "Ccs1" H 4815 5146 50  0000 L CNN
+F 1 "C" H 4815 5055 50  0000 L CNN
+F 2 "Capacitor_SMD:C_0402_1005Metric" H 4738 4950 50  0001 C CNN
+F 3 "~" H 4700 5100 50  0001 C CNN
+	1    4700 5100
 	1    0    0    -1
 $EndComp
@@
 L power:GND #PWR0107
 U 1 1 5EF2921E
-P 4700 5900
-F 0 "#PWR0107" H 4700 5650 50  0001 C CNN
-F 1 "GND" H 4705 5727 50  0000 C CNN
-F 2 "" H 4700 5900 50  0001 C CNN
-F 3 "" H 4700 5900 50  0001 C CNN
-	1    4700 5900
-	1    0    0    -1
-$EndComp
-Connection ~ 4700 5600
-Wire Wire Line
-	3150 5550 4000 5550
+P 4700 5250
+F 0 "#PWR0107" H 4700 5000 50  0001 C CNN
+F 1 "GND" H 4705 5077 50  0000 C CNN
+F 2 "" H 4700 5250 50  0001 C CNN
+F 3 "" H 4700 5250 50  0001 C CNN
+	1    4700 5250
+	1    0    0    -1
+$EndComp
 $Comp
 L Device:D D1
@@
 L Connector_Generic:Conn_01x02 J1
 U 1 1 5F0719E7
-P 1150 1500
-F 0 "J1" H 1230 1492 50  0000 L CNN
-F 1 "Conn_01x02" H 1230 1401 50  0000 L CNN
-F 2 "Connector:Banana_Jack_2Pin" H 1150 1500 50  0001 C CNN
-F 3 "~" H 1150 1500 50  0001 C CNN
-	1    1150 1500
+P 2850 2750
+F 0 "J1" H 2930 2742 50  0000 L CNN
+F 1 "Conn_01x02" H 2930 2651 50  0000 L CNN
+F 2 "Connector:Banana_Jack_2Pin" H 2850 2750 50  0001 C CNN
+F 3 "~" H 2850 2750 50  0001 C CNN
+	1    2850 2750
 	1    0    0    -1
 $EndComp
@@
 L Connector_Generic:Conn_01x02 J2
 U 1 1 5F074FA8
-P 1150 2150
-F 0 "J2" H 1230 2142 50  0000 L CNN
-F 1 "Conn_01x02" H 1230 2051 50  0000 L CNN
-F 2 "Connector:Banana_Jack_2Pin" H 1150 2150 50  0001 C CNN
-F 3 "~" H 1150 2150 50  0001 C CNN
-	1    1150 2150
+P 2850 3400
+F 0 "J2" H 2930 3392 50  0000 L CNN
+F 1 "Conn_01x02" H 2930 3301 50  0000 L CNN
+F 2 "Connector:Banana_Jack_2Pin" H 2850 3400 50  0001 C CNN
+F 3 "~" H 2850 3400 50  0001 C CNN
+	1    2850 3400
 	1    0    0    -1
 $EndComp
@@
 L Mechanical:Heatsink HS1
 U 1 1 5F0F61DC
-P 4650 2400
-F 0 "HS1" H 4792 2521 50  0000 L CNN
-F 1 "Heatsink" H 4792 2430 50  0000 L CNN
-F 2 "Heatsink:Heatsink_Stonecold_HS-132_32x14mm_2xFixation1.5mm" H 4662 2400 50  0001 C CNN
-F 3 "~" H 4662 2400 50  0001 C CNN
-	1    4650 2400
-	1    0    0    -1
-$EndComp
+P 1950 1450
+F 0 "HS1" H 2092 1571 50  0000 L CNN
+F 1 "Heatsink" H 2092 1480 50  0000 L CNN
+F 2 "Heatsink:Heatsink_Stonecold_HS-132_32x14mm_2xFixation1.5mm" H 1962 1450 50  0001 C CNN
+F 3 "~" H 1962 1450 50  0001 C CNN
+	1    1950 1450
+	1    0    0    -1
+$EndComp
+Wire Wire Line
+	4300 2900 4300 4050
+Wire Wire Line
+	4650 4700 4650 4500
+Wire Wire Line
+	4650 4500 4800 4500
+Wire Wire Line
+	4800 4500 4800 4400
+Wire Wire Line
+	4650 4850 4700 4850
+Connection ~ 4700 4850
+Wire Wire Line
+	4700 4850 4700 4950
+Wire Wire Line
+	4050 4400 3800 4400
+Wire Wire Line
+	3800 4400 3800 4300
+Wire Wire Line
+	4050 4550 3850 4550
+Wire Wire Line
+	3850 4550 3850 4950
+Wire Wire Line
+	3950 4700 4050 4700
+Wire Wire Line
+	3150 5550 3950 5550
+Wire Wire Line
+	3950 5550 3950 4700
+$Comp
+L power:GND #PWR?
+U 1 1 5EF53DE5
+P 4050 4850
+F 0 "#PWR?" H 4050 4600 50  0001 C CNN
+F 1 "GND" H 4055 4677 50  0000 C CNN
+F 2 "" H 4050 4850 50  0001 C CNN
+F 3 "" H 4050 4850 50  0001 C CNN
+	1    4050 4850
+	1    0    0    -1
+$EndComp
